File: amp.brd (EAGLE design)
At the start: 100 x 80 mm, 19 parts, among them IC1 TDA2030V

Commit message: Ádám igazításai
Parts:
- removed D3: 1N4004, diode:DO41-10
- added C8: 2000u, resistor:EB35D
- added X2, X3: (no value), con-wago-500:W237-113
- C1: value 2000uF -> 100uF; device capacitor-wima:C2.5-3 -> resistor:EB25D
- C4, C6, C7: device capacitor-wima:C2.5-3 -> resistor:E2,5-7
- C5: device capacitor-wima:C2.5-3 -> resistor:EB25D
- R7: value 4.7K -> (none); device rcl:0207/12 -> resistor:RTRIM3296W
- moved C1 170.0 mm to (-31.8, -138.4)
- moved R7 125.9 mm to (-54.6, -76.2)
- moved C5 112.7 mm to (-5.08, -91.4)
- moved C7 100.2 mm to (-1.27, -74.9)
Connections:
- net GND: now also C1.-, C4.-, C5.-, C7.-, X2.2, X3.2; no longer C4.2, C5.2, C7.2
- net N$1: now also C4.+; no longer C4.1
- net N$2: now also C8.-; no longer C1.1
- net N$3: now also C6.+; no longer C6.1
- net N$4: now also C8.+; no longer C1.2
- net N$6: now also C7.+; no longer C7.1
- net N$9: now also C6.-, R7.2; no longer C6.2, D3.A
- net VCC: now also C1.+, C5.+, X3.1; no longer C5.1
- net VPP: now also R7.3, X2.1; no longer R7.2

Commit message: some progress with brd
Parts:
- moved C1 181.8 mm to (35.6, 30.5), turned to 180 degrees
- moved R7 168.6 mm to (53.3, 53.3), turned to 90 degrees
- moved C8 154.2 mm to (78.7, 55.9)
- moved C5 133.3 mm to (74.9, 15.2), turned to 270 degrees
- moved C7 129.5 mm to (54.6, 41.9)
- moved R5 94.7 mm to (58.4, 31.8), turned to 180 degrees
- moved X2 83.7 mm to (48.3, 5.08)
- moved X3 64.9 mm to (21.6, 5.08)
- moved R6 61.6 mm to (36.8, 71.1)
- moved C3 59.5 mm to (7.62, 67.3)
- moved R2 52.4 mm to (20.3, 71.1), turned to 180 degrees
- moved C4 46.6 mm to (54.6, 16.5)
- moved X1 45.4 mm to (95.2, 31.8), turned to 90 degrees
- moved R4 39.4 mm to (17.8, 53.3), turned to 90 degrees
- moved D2 38.3 mm to (29.2, 54.6), turned to 90 degrees
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Routing:
- net GND: track 0.00 -> 269.2 mm
- net VCC: track 0.00 -> 200.8 mm
- net N$4: track 0.00 -> 137.2 mm
- net N$1: track 0.00 -> 130.8 mm
- net VPP: track 0.00 -> 114.1 mm
- net N$6: track 0.00 -> 53.2 mm
- net N$2: track 0.00 -> 34.4 mm
- net N$3: track 0.00 -> 15.2 mm
- net N$5: track 0.00 -> 9.72 mm
- net N$9: track 0.00 -> 8.89 mm

Commit message: holes added
Parts:
- added H1, H2, H3, H4: MOUNT-HOLE3.0, holes:3,0
- moved C3 4.02 mm to (6.35, 63.5)
Routing:
- net VCC: track 200.8 -> 198.1 mm
- net GND: track 269.2 -> 266.6 mm
Changed lines of the file:
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@@
 <wire x1="100" y1="80" x2="0" y2="80" width="0" layer="20"/>
 <wire x1="0" y1="80" x2="0" y2="0" width="0" layer="20"/>
-<hole x="3.81" y="76.2" drill="0.35"/>
-<hole x="3.81" y="2.54" drill="0.35"/>
-<hole x="96.52" y="2.54" drill="0.35"/>
-<hole x="96.52" y="76.2" drill="0.35"/>
 </plain>
 <attributes>
@@
 <attribute name="VALUE" x="13.081" y="16.002" size="1.27" layer="28" ratio="10" rot="MR0"/>
 </element>
-<element name="C3" library="capacitor-wima" library_urn="urn:adsk.eagle:library:116" package="C2.5-3" package3d_urn="urn:adsk.eagle:package:5436/1" value="100nF" x="7.62" y="67.31" smashed="yes">
-<attribute name="NAME" x="5.969" y="69.088" size="1.27" layer="25" ratio="10"/>
-<attribute name="VALUE" x="5.969" y="64.262" size="1.27" layer="27" ratio="10"/>
+<element name="C3" library="capacitor-wima" library_urn="urn:adsk.eagle:library:116" package="C2.5-3" package3d_urn="urn:adsk.eagle:package:5436/1" value="100nF" x="6.35" y="63.5" smashed="yes">
+<attribute name="NAME" x="4.699" y="65.278" size="1.27" layer="25" ratio="10"/>
+<attribute name="VALUE" x="4.699" y="60.452" size="1.27" layer="27" ratio="10"/>
 </element>
 <element name="C4" library="resistor" library_urn="urn:adsk.eagle:library:348" package="E2,5-7" package3d_urn="urn:adsk.eagle:package:23345/1" value="2uF" x="54.61" y="16.51" smashed="yes">
@@
 <attribute name="VALUE" x="16.0566" y="0.1524" size="1.27" layer="27" ratio="10"/>
 </element>
+<element name="H1" library="holes" library_urn="urn:adsk.eagle:library:237" package="3,0" package3d_urn="urn:adsk.eagle:package:14277/1" value="MOUNT-HOLE3.0" x="6.35" y="6.35" smashed="yes"/>
+<element name="H2" library="holes" library_urn="urn:adsk.eagle:library:237" package="3,0" package3d_urn="urn:adsk.eagle:package:14277/1" value="MOUNT-HOLE3.0" x="93.98" y="6.35" smashed="yes"/>
+<element name="H3" library="holes" library_urn="urn:adsk.eagle:library:237" package="3,0" package3d_urn="urn:adsk.eagle:package:14277/1" value="MOUNT-HOLE3.0" x="6.35" y="73.66" smashed="yes"/>
+<element name="H4" library="holes" library_urn="urn:adsk.eagle:library:237" package="3,0" package3d_urn="urn:adsk.eagle:package:14277/1" value="MOUNT-HOLE3.0" x="93.98" y="73.66" smashed="yes"/>
 </elements>
 <signals>
@@
 <contactref element="C1" pad="+"/>
 <contactref element="X3" pad="1"/>
-<wire x1="13.97" y1="71.12" x2="6.35" y2="71.12" width="0.6096" layer="1"/>
-<wire x1="6.35" y1="71.12" x2="6.35" y2="67.31" width="0.6096" layer="1"/>
+<wire x1="13.97" y1="71.12" x2="12.7" y2="71.12" width="0.6096" layer="1"/>
+<wire x1="12.7" y1="71.12" x2="5.08" y2="63.5" width="0.6096" layer="1"/>
 <wire x1="7.62" y1="30.48" x2="7.62" y2="12.78" width="0.6096" layer="1"/>
 <wire x1="7.62" y1="12.78" x2="16.59" y2="3.81" width="0.6096" layer="1"/>
@@
 <wire x1="13.97" y1="24.13" x2="7.62" y2="30.48" width="0.6096" layer="16"/>
 <wire x1="34.29" y1="24.13" x2="13.97" y2="24.13" width="0.6096" layer="16"/>
-<wire x1="6.35" y1="67.31" x2="6.35" y2="41.201975" width="0.6096" layer="1"/>
-<wire x1="6.35" y1="41.201975" x2="6.3246" y2="41.176575" width="0.6096" layer="1"/>
-<wire x1="6.3246" y1="41.176575" x2="6.3246" y2="31.7754" width="0.6096" layer="1"/>
+<wire x1="5.08" y1="63.5" x2="6.3246" y2="62.2554" width="0.6096" layer="1"/>
+<wire x1="6.3246" y1="62.2554" x2="6.3246" y2="31.7754" width="0.6096" layer="1"/>
 <wire x1="6.3246" y1="31.7754" x2="7.62" y2="30.48" width="0.6096" layer="1"/>
 <wire x1="51.3050125" y1="69.7738" x2="50.2949875" y2="69.7738" width="0.6096" layer="16"/>
@@
 <contactref element="X2" pad="2"/>
 <contactref element="C1" pad="-"/>
-<wire x1="8.89" y1="67.31" x2="8.89" y2="60.96" width="0.6096" layer="1"/>
+<wire x1="7.62" y1="63.5" x2="7.62" y2="59.69" width="0.6096" layer="1"/>
 <wire x1="8.89" y1="60.96" x2="7.62" y2="59.69" width="0.6096" layer="1"/>
 <wire x1="8.89" y1="60.96" x2="10.16" y2="59.69" width="0.6096" layer="1"/>

Commit message: Barna .brd ver2.0
Parts:
- moved H3 103.5 mm to (84.3, 5.59)
- moved H2 99.3 mm to (6.10, 52.6)
- moved C8 62.2 mm to (28.4, 19.3)
- moved C3 54.6 mm to (58.4, 47.0)
- moved C2 52.4 mm to (58.2, 42.7), flipped to the top
- moved D1 48.5 mm to (53.3, 51.8), turned to 180 degrees
- moved C4 46.0 mm to (14.2, 38.6), turned to 180 degrees
- moved X2 44.4 mm to (6.10, 19.1), turned to 270 degrees
- moved X3 36.5 mm to (6.10, 38.1), turned to 270 degrees
- moved R5 33.9 mm to (25.4, 39.4), turned to 0 degrees
- moved C6 33.4 mm to (49.5, 29.0), flipped to the top, turned to 0 degrees
- moved C1 29.0 mm to (59.4, 14.0)
- moved R6 27.0 mm to (38.1, 44.2)
- moved IC1 26.7 mm to (36.6, 57.4)
- moved D2 24.3 mm to (50.8, 43.4), turned to 270 degrees
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Connections:
- new net N$7: IC1.2, R3.1, R4.2
- net GND: no longer IC1.2, R3.1, R4.2
Routing:
- net GND: track 266.6 -> 0.00 mm
- net N$1: track 130.8 -> 16.1 mm
- net VCC: track 198.1 -> 119.9 mm, vias 0 -> 1
- net N$4: track 137.2 -> 80.2 mm, vias 0 -> 1
- net VPP: track 114.1 -> 58.7 mm
- net N$6: track 53.2 -> 20.8 mm
- net N$5: track 9.72 -> 31.9 mm, vias 0 -> 1
- net N$2: track 34.4 -> 55.5 mm
- net N$3: track 15.2 -> 30.6 mm
- net N$7: track 0.00 -> 11.7 mm
- net N$9: track 8.89 -> 9.60 mm
- added copper zone on layer 1, net GND
- added copper zone on layer 16, net GND
Other:
- board size 100 x 80 mm -> 87.8 x 56.6 mm

Commit message: final (hopefully)
Parts:
- moved X3 80.6 mm to (84.1, 17.5), turned to 90 degrees
- moved X1 77.5 mm to (6.35, 19.3), turned to 270 degrees
- moved X2 19.6 mm to (6.35, 38.6)
- turned C4 to 0 degrees
- turned C5 to 0 degrees
- turned C8 to 270 degrees
Routing:
- net N$2: track 55.5 -> 27.5 mm
- net N$4: track 80.2 -> 76.7 mm
- net VCC: track 119.9 -> 121.9 mm
- net VPP: track 58.7 -> 57.4 mm
