File: amp.sch (EAGLE design)
At the start: 2 parts

Commit message: emmegmi
Parts:
- added C1: 2000uF, capacitor-wima:C2,5-3
- added C2: 220nF, capacitor-wima:C2,5-3
- added C3: 100nF, capacitor-wima:C2,5-3
- added C4: 2uF, capacitor-wima:C2,5-3
- added C5: 100uF, capacitor-wima:C2,5-3
- added C6: 1uF, capacitor-wima:C2,5-3
- added C7: 22uF, capacitor-wima:C2,5-3
- added D1, D2: 1N4004, diode:1N4004
- added IC1: TDA2030V, linear:TDA2030V
- added R3: 150K, rcl:R-EU_0207/12
- added R4, R7: 4.7K, rcl:R-EU_0207/12
- added R5, R6: 100K, rcl:R-EU_0207/12
- added X1: (no value), con-wago-500:W237-113
- R1: value (none) -> 1; device rcl:R-US_0207/15 -> rcl:R-EU_0207/12
- R2: value 47 -> 100K
Connections:
- new net GND: C2.2, C3.2, C4.2, C5.2, C7.2, D2.A, IC1.-IN, IC1.GND, R3.1, R4.2, R5.1, R7.1, X1-2.KL
- new net N$2: C1.1, X1-1.KL
- new net N$3: C6.1, IC1.+IN, R6.2
- new net N$4: C1.2, D1.A, D2.C, IC1.OUT, R1.2, R3.2
- new net N$5: C2.1, R1.1
- new net N$6: C7.1, R2.1, R5.2, R6.1
- new net N$9: C6.2
- new net VCC: C3.1, C5.1, D1.C, IC1.V+, R2.2
- net N$1: now also C4.1, R4.1; no longer R1.2, R2.1
Other:
- moved on the sheet: R2

Commit message: terv
Parts:
- added D3: 1N4004, diode:1N4004
Connections:
- new net VPP: R7.2
- net N$9: now also D3.A
Other:
- moved on the sheet: R7
Changed lines of the file:
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@@
 <part name="GND3" library="supply1" library_urn="urn:adsk.eagle:library:371" deviceset="GND" device=""/>
 <part name="GND4" library="supply1" library_urn="urn:adsk.eagle:library:371" deviceset="GND" device=""/>
+<part name="D3" library="diode" library_urn="urn:adsk.eagle:library:210" deviceset="1N4004" device="" package3d_urn="urn:adsk.eagle:package:43336/1"/>
+<part name="SUPPLY2" library="supply2" library_urn="urn:adsk.eagle:library:372" deviceset="VPP" device=""/>
 </parts>
 <sheets>
@@
 <attribute name="VALUE" x="-46.736" y="41.021" size="1.778" layer="96"/>
 </instance>
-<instance part="R7" gate="G$1" x="-63.5" y="76.2" smashed="yes" rot="R90">
-<attribute name="NAME" x="-67.5386" y="77.47" size="1.778" layer="95" rot="R180"/>
-<attribute name="VALUE" x="-57.658" y="77.47" size="1.778" layer="96" rot="R180"/>
+<instance part="R7" gate="G$1" x="-60.96" y="73.66" smashed="yes" rot="R90">
+<attribute name="NAME" x="-62.4586" y="74.93" size="1.778" layer="95" rot="R180"/>
+<attribute name="VALUE" x="-62.738" y="72.39" size="1.778" layer="96" rot="R180"/>
 </instance>
 <instance part="SUPPLY1" gate="G$1" x="33.02" y="104.14" smashed="yes" rot="R270">
@@
 <attribute name="VALUE" x="50.8" y="10.16" size="1.778" layer="96"/>
 </instance>
-<instance part="GND2" gate="1" x="-63.5" y="58.42" smashed="yes">
-<attribute name="VALUE" x="-66.04" y="55.88" size="1.778" layer="96"/>
+<instance part="GND2" gate="1" x="-60.96" y="58.42" smashed="yes">
+<attribute name="VALUE" x="-63.5" y="55.88" size="1.778" layer="96"/>
 </instance>
 <instance part="GND3" gate="1" x="12.7" y="88.9" smashed="yes">
@@
 <instance part="GND4" gate="1" x="25.4" y="88.9" smashed="yes">
 <attribute name="VALUE" x="22.86" y="86.36" size="1.778" layer="96"/>
+</instance>
+<instance part="D3" gate="1" x="-58.42" y="73.66" smashed="yes" rot="MR0">
+<attribute name="NAME" x="-55.88" y="76.6826" size="1.778" layer="95"/>
+<attribute name="VALUE" x="-48.26" y="68.8086" size="1.778" layer="96" rot="MR0"/>
+</instance>
+<instance part="SUPPLY2" gate="G$1" x="-60.96" y="81.28" smashed="yes">
+<attribute name="VALUE" x="-62.865" y="84.455" size="1.778" layer="96"/>
 </instance>
 </instances>
@@
 <pinref part="C6" gate="G$1" pin="2"/>
 <wire x1="-30.48" y1="73.66" x2="-55.88" y2="73.66" width="0.1524" layer="91"/>
+<pinref part="D3" gate="1" pin="A"/>
 </segment>
 </net>
@@
 <segment>
 <pinref part="R7" gate="G$1" pin="1"/>
-<wire x1="-63.5" y1="71.12" x2="-63.5" y2="60.96" width="0.1524" layer="91"/>
+<wire x1="-60.96" y1="68.58" x2="-60.96" y2="60.96" width="0.1524" layer="91"/>
 <pinref part="GND2" gate="1" pin="GND"/>
 </segment>
@@
 </segment>
 </net>
+<net name="VPP" class="0">
+<segment>
+<pinref part="R7" gate="G$1" pin="2"/>
+<pinref part="SUPPLY2" gate="G$1" pin="VPP"/>
+</segment>
+</net>

Commit message: Ádám igazításai
Parts:
- removed D3: 1N4004, diode:1N4004
- added C8: 2000u, resistor:CPOL-EUE10-35
- added X2, X3: (no value), con-wago-500:W237-113
- C1: value 2000uF -> 100uF; device capacitor-wima:C2,5-3 -> resistor:CPOL-EUE10-25
- C4, C6, C7: device capacitor-wima:C2,5-3 -> resistor:CPOL-EUE2.5-7
- C5: device capacitor-wima:C2,5-3 -> resistor:CPOL-EUE10-25
- R7: value 4.7K -> (none); device rcl:R-EU_0207/12 -> resistor:R-TRIMM3296W
Connections:
- net GND: now also C1.-, C4.-, C5.-, C7.-, R7.A, X2-2.KL, X3-2.KL; no longer C4.2, C5.2, C7.2, R7.1
- net N$1: now also C4.+; no longer C4.1
- net N$2: now also C8.-; no longer C1.1
- net N$3: now also C6.+; no longer C6.1
- net N$4: now also C8.+; no longer C1.2
- net N$6: now also C7.+; no longer C7.1
- net N$9: now also C6.-, R7.S; no longer C6.2, D3.A
- net VCC: now also C1.+, C5.+, X3-1.KL; no longer C5.1
- net VPP: now also R7.E, X2-1.KL; no longer R7.2

Commit message: final (hopefully)
Parts:
- added H1, H2, H3, H4: MOUNT-HOLE3.0, holes:MOUNT-HOLE3.0
Connections:
- new net N$7: IC1.-IN, R3.1, R4.2
- net GND: no longer IC1.-IN, R3.1, R4.2
